Commit message: Added updated tello urdf and meshes

File: tello_description/urdf/generic_camera.urdf.xacro (robot description, xacro)
@@ -1,4 +1,4 @@
 <?xml version="1.0"?>
-<robot xmlns:xacro="http://ros.org/wiki/xacro">
+<robot xmlns:xacro="http://www.ros.org/wiki/xacro">
   <xacro:property name="M_PI" value="3.1415926535897931" />
   <xacro:macro name="generic_camera" params="name parent *origin ros_topic cam_info_topic update_rate res_x res_y image_format hfov">
@@ -31,5 +31,5 @@
     </link>
     <joint name="${name}_optical_joint" type="fixed">
-      <origin xyz="0 0 0" rpy="${-M_PI/2} 0.0 ${-M_PI/2}" />
+      <origin xyz="0 0 0" rpy="0.0 0.0 0.0" />
       <parent link="${name}_link" />
       <child link="${name}_optical_frame"/>
@@ -50,9 +50,4 @@
             <far>100</far>
           </clip>
-	  <!--noise>
-		  <type>gaussian</type>
-		  <mean>0.0</mean>
-		  <stddev>0.007</stddev>
-	  </noise-->
         </camera>
         <plugin name="${name}_camera_controller" filename="libgazebo_ros_camera.so">
@@ -60,12 +55,10 @@
           <imageTopicName>${ros_topic}</imageTopicName>
           <cameraInfoTopicName>${cam_info_topic}</cameraInfoTopicName>
-	  <frameName>${name}_optical_frame</frameName>
-	  <!--hackBaseline>0.07</hackBaseline>
-          <Cx>526.857585</Cx>
-	  <Cy>305.59503</Cy>
-	  <distortionK1>-0.136594</distortionK1>
-          <distortionK2>0.179016</distortionK2>
-          <distortionT1>-0.019119</distortionT1>
-          <distortionT2>0.012205</distortionT2-->
+          <frameName>${name}_optical_frame</frameName>
+          <distortionK1>0.0</distortionK1>
+          <distortionK2>0.0</distortionK2>
+          <distortionK3>0.0</distortionK3>
+          <distortionT1>0.0</distortionT1>
+          <distortionT2>0.0</distortionT2>
         </plugin>
       </sensor>

File: tello_description/urdf/tello.gazebo.xacro (robot description, xacro)
@@ -1,5 +1,5 @@
 <?xml version="1.0"?>
 <robot name="quadrotor" xmlns:xacro="http://www.ros.org/wiki/xacro">
-    <xacro:include filename="$(find tello_description)/urdf/quadrotor_with_cam.urdf.xacro" />
+    <xacro:include filename="$(find tello_description)/urdf/tello.urdf.xacro" />
     <xacro:include filename="$(find hector_quadrotor_gazebo)/urdf/quadrotor_plugins.gazebo.xacro" />
 </robot>

File: tello_description/urdf/tello.urdf.xacro (robot description, xacro)
@@ -1,6 +1,16 @@
 <?xml version="1.0"?>
-<robot xmlns:xacro="http://www.ros.org/wiki/xacro">
-  <xacro:include filename="$(find hector_sensors_description)/urdf/sonar_sensor.urdf.xacro" />
-  <xacro:property name="pi" value="3.1415926535897931" />
+<robot name="quadrotor" xmlns:xacro="http://www.ros.org/wiki/xacro">
+  <xacro:property name="M_PI" value="3.1415926535897931" />
+  <!-- <link name="world" />
+  <joint name="world_to_new_world_joint=" type="fixed">
+    <origin xyz="0 0 0" rpy="1.57 0.0 0.0" />
+    <parent link="world"/>
+    <child link="new_world"/>
+  </joint>
+  <link name="new_world" />
+  <joint name="new_world_to_base_joint=" type="fixed">
+    <parent link="new_world"/>
+    <child link="base_link"/>
+  </joint> -->
   <!-- Main quadrotor link -->
   <xacro:macro name="quadrotor_base_macro">
@@ -8,24 +18,35 @@
       <inertial>
         <mass value="0.085" />
-        <origin xyz="0 0 0" />
+        <origin xyz="0 0 0" rpy="0 0 ${-M_PI/2}" />
         <inertia ixx="0.01152" ixy="0.0" ixz="0.0" iyy="0.01152" iyz="0.0" izz="0.0218" />
       </inertial>
       <visual>
-        <origin xyz="0 0 0" rpy="0 0 0" />
+        <origin xyz="0 0 0" rpy="0 0 ${-M_PI/2}" />
         <geometry>
-	  <mesh filename="package://tello_description/meshes/tello.dae"/>
+          <!--3d model of Ryze Tello drone provided by https://www.halfchrome.com/downloads/dji-tello-cad-model/-->
+	        <mesh filename="package://tello_description/meshes/tello.dae"/>
         </geometry>
       </visual>
       <collision>
-        <origin xyz="0 0 0" rpy="0 0 0" />
+        <origin xyz="0 0 0" rpy="0 0 ${-M_PI/2}" />
         <geometry>
-	  <mesh filename="package://tello_description/meshes/tello.stl"/>
+          <!--3d model of Ryze Tello drone provided by https://www.halfchrome.com/downloads/dji-tello-cad-model/-->
+	        <mesh filename="package://tello_description/meshes/tello.stl"/>
         </geometry>
       </collision>
     </link>
-    <!-- Sonar height sensor -->
-    <xacro:sonar_sensor name="sonar" parent="base_link" ros_topic="sonar_height" update_rate="10" min_range="0.03" max_range="3.0" field_of_view="${40*pi/180}" ray_count="3">
-      <origin xyz="-0.01 0.0 0.005" rpy="0 ${90*pi/180} 0"/>
+    <!-- Altitude sensor. Tello uses a pair of IR sensors instead, but we couldn't find any in hector_sensors package -->
+    <xacro:include filename="$(find tello_description)/urdf/sonar_sensor.urdf.xacro" />
+    <xacro:sonar_sensor name="sonar" parent="base_link" ros_topic="sonar_height" update_rate="10" min_range="0.03" max_range="3.0" field_of_view="${10*pi/180}" ray_count="1">
+      <origin xyz="-0.02 0.0 0.025" rpy="0 1.5707 0"/>
     </xacro:sonar_sensor>
+    <!--Front camera. With real Tello there is no way to access downward looking camera-->
+        <!-- Forward facing camera -->
+    <xacro:include filename="$(find tello_description)/urdf/generic_camera.urdf.xacro" />
+    <xacro:generic_camera name="front_cam" parent="base_link" ros_topic="camera/image" cam_info_topic="camera/camera_info" res_x="640" res_y="480" image_format="R8G8B8" update_rate="60" hfov="83">
+      <origin xyz="0.07 0.00 0.03" rpy="0 0 0"/>
+    </xacro:generic_camera>
   </xacro:macro>
+  <!--Base of the hector_quadrotor, which connects gazebo plugins and flight controller from the hector_quadrotor package-->
+  <xacro:quadrotor_base_macro />
 </robot>
